File: hardware/Business Card v2.kicad_pcb (KiCad board)
At the start: 2 copper layers, 85.4 x 54.1 mm, 39 parts, among them J1 Conn_01x03_Pin, Q1 DMP21D0UFB4-P, U1 ATTINY816-MNR, U3 NT3H2111W0FHKH

Commit message: Amber LEDs, R4 BOM fix, JLCPCB fab outputs
- LED1-LED20: red XL-1608SURC-06FJ (C7371900) -> amber XL-1608UYC-06FJ (C7371901), the same
  family and 600 mcd brightness, copied field-for-field from LED22. The footprint is unchanged:
  both land patterns put the cathode on the -x pad. Phosphor-green C965805 was rejected
  (60 mcd, 10x dimmer on NFC power).
- R4 lacked an LCSC number in the original (JLCPCB would leave it unplaced); it now has C25076
  like R1/R5-R7.
- Both are applied deterministically: board via apply_final.py, schematic via tools/bom/leds.py,
  each regenerated from 57a460f.
- tools/fab/make_fab.sh -> fab/gerbers.zip, bom_jlc.csv, cpl_jlc.csv (37 parts).
- Verified with kicad-cli 10.0.6. DRC with schematic parity 45->45 and ERC 106->106, identical
  per category to the original. Silk round-trip: only silk changed, 0 DFM errors, QR decodes.

Co-Authored-By: Claude Opus 5.5 (1M context) <noreply@anthropic.com>
Parts:
- LED1, LED10, LED11, LED12, LED13, LED14, LED15, LED16, LED17, LED18, LED19, LED2, LED20, LED3, LED4, LED5, LED6, LED7, LED8, LED9: value XL-1608SURC-06FJ -> XL-1608UYC-06FJ
