File: hardware/Business Card v2.kicad_sch (KiCad schematic)
At the start: 39 parts, among them J1 Conn_01x03_Pin, Q1 DMP21D0UFB4-P, U1 ATTINY816-MNR, U3 NT3H2111W0FHKH

Commit message: Amber LEDs, R4 BOM fix, JLCPCB fab outputs
- LED1-LED20: red XL-1608SURC-06FJ (C7371900) -> amber XL-1608UYC-06FJ (C7371901), the same
  family and 600 mcd brightness, copied field-for-field from LED22. The footprint is unchanged:
  both land patterns put the cathode on the -x pad. Phosphor-green C965805 was rejected
  (60 mcd, 10x dimmer on NFC power).
- R4 lacked an LCSC number in the original (JLCPCB would leave it unplaced); it now has C25076
  like R1/R5-R7.
- Both are applied deterministically: board via apply_final.py, schematic via tools/bom/leds.py,
  each regenerated from 57a460f.
- tools/fab/make_fab.sh -> fab/gerbers.zip, bom_jlc.csv, cpl_jlc.csv (37 parts).
- Verified with kicad-cli 10.0.6. DRC with schematic parity 45->45 and ERC 106->106, identical
  per category to the original. Silk round-trip: only silk changed, 0 DFM errors, QR decodes.

Co-Authored-By: Claude Opus 5.5 (1M context) <noreply@anthropic.com>
Parts:
- LED1, LED10, LED11, LED12, LED13, LED14, LED15, LED16, LED17, LED18, LED19, LED2, LED20, LED3, LED4, LED5, LED6, LED7, LED8, LED9: value XL-1608SURC-06FJ -> XL-1608UYC-06FJ; LCSC C7371900 -> C7371901; Manufacturer Part XL-1608SURC-06FJ -> XL-1608UYC-06FJ
- R4: LCSC (none) -> C25076

Commit message: BOM: C1 is the 0402 part (C1552), one BOM line per LCSC part
- C1 (1.5 pF antenna tuning cap, 0402 footprint) carried C1639, which is 0603CG1R5C500NT, an
  0603 part. JLCPCB matched it as an 0603. It is now C1552 (0402CG1R5C500NT), the same FH C0G
  part in 0402; 221k in stock. Applied via tools/bom/fixes.py to both board and schematic.
- make_fab.sh merges rows that share an LCSC number, so LED1-20 + LED22 (one part on two
  footprint names) are one line. JLCPCB had left both lines Unconfirmed at qty 0.
- Re-verified: DRC with parity 45->45 and ERC 106->106, identical per category; 37 parts placed.

Co-Authored-By: Claude Opus 5.5 (1M context) <noreply@anthropic.com>
Parts:
- C1: LCSC C1639 -> C1552
Changed lines of the file:
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@@
 			)
 		)
-		(property "LCSC" "C1639"
+		(property "LCSC" "C1552"
 			(at 49.53 49.53 0)
 			(effects
